File: hardware/DashShield/DashShield.kicad_sch (KiCad schematic)
At the start: 10 parts, among them J1 GPIO, U1 CAT24C256, U2 MCP2562-E-SN, U3 MCP2562-E-SN, U4 MCP2515-xST, U5 MCP2515-xST

Commit message: feat: initial CAN interfaces
Parts:
- removed U3: MCP2562-E-SN, Package_SO:SOIC-8_3.9x4.9mm_P1.27mm, symbol Interface_CAN_LIN:MCP2562-E-SN
- removed U5: MCP2515-xST, Package_SO:TSSOP-20_4.4x6.5mm_P0.65mm, symbol Interface_CAN_LIN:MCP2515-xST
- added C10, C11, C2, C3, C6, C7: 100nF, symbol Device:C
- added C12, C13: 10F, symbol Device:C_Polarized
- added C4, C5, C8, C9: 22pF, symbol Device:C
- added D1: 5.1V, symbol Device:D_Zener
- added D2, D3: 2.7V, symbol Device:D_Zener
- added D4: LED, symbol Device:LED
- added D5: CRS15, Diode_SMD:D_SOD-123F, symbol Device:D
- added J2: Steering Wheel, symbol Connector_Generic:Conn_02x06_Counter_Clockwise
- added J3: Dash LEDs, symbol Connector_Generic:Conn_02x04_Counter_Clockwise
- added J4: CAN 0, symbol Connector_Generic_Shielded:Conn_01x02_Shielded
- added J5: PWR, symbol Connector_Generic:Conn_01x02
- added J6: CAN 1, symbol Connector_Generic_Shielded:Conn_01x02_Shielded
- added JP2, JP5: Termination Jumper, symbol Jumper:Jumper_2_Open
- added JP3, JP4: Shielding Jumper, symbol Jumper:Jumper_2_Open
- added Q1, Q2, Q3, Q4, Q5, Q6: 2N7002, Package_TO_SOT_SMD:SOT-23, symbol Transistor_FET:2N7002
- added R10, R12: 0, symbol Device:R
- added R11, R13: 4k7, symbol Device:R
- added R14, R9: 120, symbol Device:R
- added R15, R17, R19: 1k, symbol Device:R
- added R16: 3.3Ω, symbol Device:R
- added R3, R4, R5, R6, R7, R8: 270, symbol Device:R
- added U3: MCP2515-xST, Package_SO:TSSOP-20_4.4x6.5mm_P0.65mm, symbol Interface_CAN_LIN:MCP2515-xST
- added U5: MCP2562-E-SN, Package_SO:SOIC-8_3.9x4.9mm_P1.27mm, symbol Interface_CAN_LIN:MCP2562-E-SN
- added Y1, Y2: 8MHz, symbol Device:Crystal
Connections:
- net +5V: now also U2.3 (VDD), C10.1, C3.1, J3.1 (Pin_1), J3.8 (Pin_8), U5.3 (VDD)
- net GND: now also U2.2 (VSS), U2.8 (STBY), U4.10 (VSS), C10.2, C11.2, C13.2, C2.2, C3.2, C4.2, C5.1, C6.2, C7.2, C8.2, C9.1, D1.2 (A), D3.2 (A), D4.1 (K), J5.2 (Pin_2), JP3.1 (A), JP4.1 (A), Q1.2 (S), Q2.2 (S), Q3.2 (S), Q4.2 (S), Q5.2 (S), Q6.2 (S), R11.2, R13.2, R17.1, U3.10 (VSS), U5.2 (VSS), U5.8 (STBY)
- net GPIO10/SPI0.MOSI: now also U4.16 (SI), U3.16 (SI)
- net GPIO11/SPI0.SCLK: now also U4.14 (SCK), U3.14 (SCK)
- net GPIO7/SPI0.CE1: now also U3.18 (~{CS})
- net GPIO8/SPI0.CE0: now also U4.18 (~{CS})
- net GPIO9/SPI0.MISO: now also U4.17 (SO), U3.17 (SO)
- net CAN0 TX: now reaches U4.1 (TXCAN)
- net CAN0 TX: now also U2.1 (TXD)
- net CAN0 INT: now reaches U4.13 (~{INT})
- net at U4.19 (~{RESET}): now also R11.1
- net CAN0 RX: now reaches U4.2 (RXCAN)
- net CAN0 RX: now also U2.4 (RXD)
- net +3.3V: now reaches U4.20 (VDD)
- net +3.3V: now also U2.5 (Vio), C11.1, C2.1, C6.1, C7.1, U3.20 (VDD), U5.5 (Vio)
- net at U4.8 (OSC2): now also R10.2
- net at U4.9 (OSC1): now also C5.2, Y1.1
- net CAN0 Low: now reaches U2.6 (CANL)
- net CAN0 Low: now also J4.2 (Pin_2), JP2.2 (B)
- net CAN0 High: now reaches U2.7 (CANH)
- net CAN0 High: now also J4.1 (Pin_1), R9.1
- new net: JP2.1 (A), R9.2
- new net: Q2.3 (D), R4.2
- new net: C12.2, C13.1, D2.2 (A), D3.1 (K), R15.1, R17.2
- new net: C8.1, R12.1, Y2.2
- new net: R12.2, U3.8 (OSC2)
- new net: C12.1, D2.1 (K), D5.2 (A), R15.2, R16.1, R19.2
- new net: J4.SH (Shield), JP3.2 (B)
- new net: D4.2 (A), R19.1
- new net: Q5.3 (D), R7.2
- new net: C4.1, R10.1, Y1.2
- new net: JP5.1 (A), R14.2
- new net: C9.2, U3.9 (OSC1), Y2.1
- new net: Q1.3 (D), R3.2
- new net: R13.1, U3.19 (~{RESET})
- new net: Q3.3 (D), R5.2
- new net: Q4.3 (D), R6.2
- new net: Q6.3 (D), R8.2
- new net: J6.SH (Shield), JP4.2 (B)
- new net CAN1 High: J6.1 (Pin_1), R14.1, U5.7 (CANH)
- new net CAN1 INT: U3.13 (~{INT})
- new net CAN1 Low: J6.2 (Pin_2), JP5.2 (B), U5.6 (CANL)
- new net CAN1 RX: U3.2 (RXCAN), U5.4 (RXD)
- new net CAN1 TX: U3.1 (TXCAN), U5.1 (TXD)
- new net FAST 0: Q4.1 (G)
- new net FAST 1: Q5.1 (G)
- new net FAST 2: Q6.1 (G)
- new net FAST LED 0: J3.7 (Pin_7), R6.1
- new net FAST LED 1: J3.6 (Pin_6), R7.1
- new net FAST LED 2: J3.5 (Pin_5), R8.1
- new net SLOW 0: Q1.1 (G)
- new net SLOW 1: Q2.1 (G)
- new net SLOW 2: Q3.1 (G)
- new net SLOW LED 0: J3.2 (Pin_2), R3.1
- new net SLOW LED 1: J3.3 (Pin_3), R4.1
- new net SLOW LED 2: J3.4 (Pin_4), R5.1
- new net VS: D1.1 (K), D5.1 (K), J5.1 (Pin_1), R16.2
- no-connect marks 3 -> 15
Other:
- note added: "CAN0 Controller"
- note added: "CAN0 Network"
- note added: "CAN0 Transceiver"
- note added: "CAN1 Controller"
- note added: "CAN1 Network"
- note added: "CAN1 Transceiver"
- note added: "Dash Energy Usage/Lap Time LEDs"
- note added: "HAT EEPROM"
- note added: "Pi Header"
- note added: "Power Distribution"
- note removed: "Additional pin functions: https://pinout.xyz/"
- moved on the sheet: C1, J1, JP1, R1, R2, U1, U2, U4
