File: hardware/DashShield.kicad_pcb (KiCad board)
At the start: 2 copper layers, 65 x 30 mm, 5 parts, among them J1 GPIO

Commit message: feat: initial revision of dash PCB schematic
Parts:
- removed MH1, MH2, MH3, MH4: MountingHole_2.7mm_M2.5, MountingHole:MountingHole_2.7mm_M2.5
- added C1: 100n, Capacitor_SMD:C_0603_1608Metric, F.Cu at (73.5, 118.0)
- added C10: 100nF, Capacitor_SMD:C_0603_1608Metric, F.Cu at (73.5, 140.5)
- added C11: 100nF, Capacitor_SMD:C_0603_1608Metric, F.Cu at (77.5, 118.0)
- added C12: 25F, Capacitor_THT:CP_Radial_D16.0mm_P7.50mm, F.Cu at (39.0, 100.3)
- added C13: 25F, Capacitor_THT:CP_Radial_D16.0mm_P7.50mm, F.Cu at (59.0, 143.0)
- added C14: 10uF, Capacitor_SMD:C_0603_1608Metric, F.Cu at (77.5, 120.5)
- added C15: 10uF, Capacitor_SMD:C_0603_1608Metric, F.Cu at (77.5, 123.0)
- added C16: 10uF, Capacitor_SMD:C_0603_1608Metric, F.Cu at (77.5, 125.5)
- added C17: 100nF, Capacitor_SMD:C_0603_1608Metric, F.Cu at (77.5, 128.0)
- added C18: 100nF, Capacitor_SMD:C_0603_1608Metric, F.Cu at (77.5, 130.5)
- added C19: 10uF, Capacitor_SMD:C_0603_1608Metric, F.Cu at (77.5, 133.0)
- added C2: 100nF, Capacitor_SMD:C_0603_1608Metric, F.Cu at (73.5, 120.5)
- added C20: 10nF, Capacitor_SMD:C_0603_1608Metric, F.Cu at (77.5, 135.5)
- added C21: 10nF, Capacitor_SMD:C_0603_1608Metric, F.Cu at (77.5, 138.0)
- added C22: 10nF, Capacitor_SMD:C_0603_1608Metric, F.Cu at (77.5, 140.5)
- added C3: 100nF, Capacitor_SMD:C_0603_1608Metric, F.Cu at (73.5, 123.0)
- added C4: 22pF, Capacitor_SMD:C_0603_1608Metric, F.Cu at (73.5, 125.5)
- added C5: 22pF, Capacitor_SMD:C_0603_1608Metric, F.Cu at (73.5, 128.0)
- added C6: 100nF, Capacitor_SMD:C_0603_1608Metric, F.Cu at (73.5, 130.5)
- added C7: 100nF, Capacitor_SMD:C_0603_1608Metric, F.Cu at (73.5, 133.0)
- added C8: 22pF, Capacitor_SMD:C_0603_1608Metric, F.Cu at (73.5, 135.5)
- added C9: 22pF, Capacitor_SMD:C_0603_1608Metric, F.Cu at (73.5, 138.0)
- added D1: 5.1V, Diode_SMD:D_SMA, F.Cu at (85.1, 104.4)
- added D2: 2.7V, Package_TO_SOT_SMD:SOT-23, F.Cu at (78.4, 104.4)
- added D3: 2.7V, Package_TO_SOT_SMD:SOT-23, F.Cu at (71.1, 109.9)
- added D4: LED, LED_SMD:LED_0603_1608Metric, F.Cu at (97.6, 138.0)
- added D5: CRS15, Diode_SMD:D_SOD-123F, F.Cu at (98.3, 131.7)
- added D6: CRS15, Diode_SMD:D_SOD-123F, F.Cu at (98.3, 135.1)
- added J2: Steering Wheel, Connector_Molex:Molex_Micro-Fit_3.0_43045-1212_2x06_P3.00mm_Vertical, F.Cu at (75.8, 145.3)
- added J3: Dash LEDs, Connector_Molex:Molex_Micro-Fit_3.0_43045-0812_2x04_P3.00mm_Vertical, F.Cu at (84.3, 156.1)
- added J4: CAN0, Connector_Molex:Molex_Micro-Fit_3.0_43650-0315_1x03_P3.00mm_Vertical, F.Cu at (57.8, 155.3)
- added J5: PWR, Connector_Molex:Molex_Micro-Fit_3.0_43650-0215_1x02_P3.00mm_Vertical, F.Cu at (116.4, 153.7)
- added J7: CAN1, Connector_Molex:Molex_Micro-Fit_3.0_43650-0315_1x03_P3.00mm_Vertical, F.Cu at (57.8, 163.1)
- added JP1: WP Enable Jumper, Connector_PinHeader_2.54mm:PinHeader_1x02_P2.54mm_Vertical, F.Cu at (117.3, 136.5)
- added JP2: Termination Jumper, Connector_PinHeader_2.54mm:PinHeader_1x02_P2.54mm_Vertical, F.Cu at (121.9, 136.5)
- added JP3: Shielding Jumper, Connector_PinHeader_2.54mm:PinHeader_1x02_P2.54mm_Vertical, F.Cu at (126.6, 136.5)
- added JP4: Shielding Jumper, Connector_PinHeader_2.54mm:PinHeader_1x02_P2.54mm_Vertical, F.Cu at (131.2, 136.5)
- added JP5: Termination Jumper, Connector_PinHeader_2.54mm:PinHeader_1x02_P2.54mm_Vertical, F.Cu at (135.9, 136.5)
- added Q1: 2N7002, Package_TO_SOT_SMD:SOT-23, F.Cu at (98.0, 118.9)
- added Q2: 2N7002, Package_TO_SOT_SMD:SOT-23, F.Cu at (98.0, 123.4)
- added Q3: 2N7002, Package_TO_SOT_SMD:SOT-23, F.Cu at (98.0, 127.8)
- added Q4: 2N7002, Package_TO_SOT_SMD:SOT-23, F.Cu at (102.9, 118.9)
- added Q5: 2N7002, Package_TO_SOT_SMD:SOT-23, F.Cu at (102.9, 123.4)
- added Q6: 2N7002, Package_TO_SOT_SMD:SOT-23, F.Cu at (102.9, 127.8)
- added Q7: 2N7002, Package_TO_SOT_SMD:SOT-23, F.Cu at (107.8, 118.9)
- added Q8: 2N7002, Package_TO_SOT_SMD:SOT-23, F.Cu at (107.8, 123.4)
- added Q9: 2N7002, Package_TO_SOT_SMD:SOT-23, F.Cu at (107.8, 127.8)
- added R1: 3.9k, Resistor_SMD:R_0603_1608Metric, F.Cu at (81.5, 118.0)
- added R10: 0, Resistor_SMD:R_0603_1608Metric, F.Cu at (81.5, 140.5)
- added R11: 4k7, Resistor_SMD:R_0603_1608Metric, F.Cu at (85.5, 118.0)
- added R12: 0, Resistor_SMD:R_0603_1608Metric, F.Cu at (85.5, 120.5)
- added R13: 4k7, Resistor_SMD:R_0603_1608Metric, F.Cu at (85.5, 123.0)
- added R14: 120, Resistor_SMD:R_0603_1608Metric, F.Cu at (85.5, 125.5)
- added R15: 1k, Resistor_SMD:R_0603_1608Metric, F.Cu at (85.5, 128.0)
- added R16: 3.3, Resistor_SMD:R_0603_1608Metric, F.Cu at (85.5, 130.5)
- added R17: 1k, Resistor_SMD:R_0603_1608Metric, F.Cu at (85.5, 133.0)
- added R18: 20k, Resistor_SMD:R_0603_1608Metric, F.Cu at (85.5, 135.5)
- added R19: 1k, Resistor_SMD:R_0603_1608Metric, F.Cu at (85.5, 138.0)
- added R2: 3.9k, Resistor_SMD:R_0603_1608Metric, F.Cu at (81.5, 120.5)
- added R20: 10k, Resistor_SMD:R_0603_1608Metric, F.Cu at (85.5, 140.5)
- added R21: 10k, Resistor_SMD:R_0603_1608Metric, F.Cu at (89.5, 118.0)
- added R22: 20k, Resistor_SMD:R_0603_1608Metric, F.Cu at (89.5, 120.5)
- added R23: 270, Resistor_SMD:R_0603_1608Metric, F.Cu at (89.5, 123.0)
- added R24: 270, Resistor_SMD:R_0603_1608Metric, F.Cu at (89.5, 125.5)
- added R25: 270, Resistor_SMD:R_0603_1608Metric, F.Cu at (89.5, 128.0)
- added R26: 270, Resistor_SMD:R_0603_1608Metric, F.Cu at (89.5, 130.5)
- added R27: 270, Resistor_SMD:R_0603_1608Metric, F.Cu at (89.5, 133.0)
- added R28: 270, Resistor_SMD:R_0603_1608Metric, F.Cu at (89.5, 135.5)
- added R29: 1k, Resistor_SMD:R_0603_1608Metric, F.Cu at (89.5, 138.0)
- added R3: 270, Resistor_SMD:R_0603_1608Metric, F.Cu at (81.5, 123.0)
- added R30: 1k, Resistor_SMD:R_0603_1608Metric, F.Cu at (89.5, 140.5)
- added R31: 10k, Resistor_SMD:R_0603_1608Metric, F.Cu at (93.5, 118.0)
- added R32: 10k, Resistor_SMD:R_0603_1608Metric, F.Cu at (93.5, 120.5)
- added R33: 1k, Resistor_SMD:R_0603_1608Metric, F.Cu at (83.0, 108.0)
- added R35: 10k, Resistor_SMD:R_0603_1608Metric, F.Cu at (93.5, 123.0)
- added R36: 10k, Resistor_SMD:R_0603_1608Metric, F.Cu at (93.5, 125.5)
- added R37: 10k, Resistor_SMD:R_0603_1608Metric, F.Cu at (93.5, 128.0)
- added R38: 10k, Resistor_SMD:R_0603_1608Metric, F.Cu at (93.5, 130.5)
- added R39: 10k, Resistor_SMD:R_0603_1608Metric, F.Cu at (93.5, 133.0)
- added R4: 270, Resistor_SMD:R_0603_1608Metric, F.Cu at (81.5, 125.5)
- added R40: 10k, Resistor_SMD:R_0603_1608Metric, F.Cu at (93.5, 135.5)
- added R5: 270, Resistor_SMD:R_0603_1608Metric, F.Cu at (81.5, 128.0)
- added R6: 270, Resistor_SMD:R_0603_1608Metric, F.Cu at (81.5, 130.5)
- added R7: 270, Resistor_SMD:R_0603_1608Metric, F.Cu at (81.5, 133.0)
- added R8: 270, Resistor_SMD:R_0603_1608Metric, F.Cu at (81.5, 135.5)
- added R9: 120, Resistor_SMD:R_0603_1608Metric, F.Cu at (81.5, 138.0)
- added U1: CAT24C256, Package_SO:SOIC-8_3.9x4.9mm_P1.27mm, F.Cu at (75.7, 155.8)
- added U2: MCP2562-E-SN, Package_SO:SOIC-8_3.9x4.9mm_P1.27mm, F.Cu at (75.7, 162.3)
- added U3: MCP2515-xST, Package_SO:TSSOP-20_4.4x6.5mm_P0.65mm, F.Cu at (100.6, 167.5)
- added U4: MCP2515-xST, Package_SO:TSSOP-20_4.4x6.5mm_P0.65mm, F.Cu at (100.6, 175.5)
- added U5: MCP2562-E-SN, Package_SO:SOIC-8_3.9x4.9mm_P1.27mm, F.Cu at (75.7, 168.7)
- added U6: ~, U3V40x:U3V40x, F.Cu at (88.1, 171.6)
- added Y1: 8MHz, Crystal:Crystal_SMD_HC49-SD, F.Cu at (60.8, 170.6)
- added Y2: 8MHz, Crystal:Crystal_SMD_HC49-SD, F.Cu at (60.8, 176.8)
- J1: moved to F.Cu
- moved J1 44.8 mm to (64.1, 81.9), turned to 90 degrees
Connections:
- J1 pad 18: /GPIO24 -> /CAN0 INT
- J1 pad 22: /GPIO25 -> /CAN1 INT
- J1 pad 29: /GPIO5 -> /FAST 0
- J1 pad 31: /GPIO6 -> /FAST 1
- J1 pad 32: /GPIO12/PWM0 -> /FAST 2
Other:
- board outline removed
- board text removed: "Extend PCB edge 0.5mm if using SMT header"
- board text removed: "PoE"
